File: hardware/01_PoE_Frontend.kicad_sch (KiCad schematic)
At the start: 0 parts

Commit message: Add gh0stee.com branding to all title blocks and README
Added (company "gh0stee.com") to the KiCad title_block of all six
schematics (root + Sheets 01–05) and the PCB file so the company name
appears in every printed/exported title block. Added a byline link to
README.md below the project description.

Co-Authored-By: Claude Sonnet 4.6 <noreply@anthropic.com>
Other:
- company: (none) -> gh0stee.com
Changed lines of the file:
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@@
 		(date "2026-05-10")
 		(rev "A")
+		(company "gh0stee.com")
 		(comment 1 "RJ45 + integrated magnetics, ESD protection, MDI breakout")
 		(comment 2 "PoE pair-set center taps to PD converter (sheet 02)")
