File: hardware/02_PoE_PD_Converter.kicad_sch (KiCad schematic)
At the start: 0 parts

Commit message: Fix four doc inconsistencies found in project review
- README spec table: 22 kΩ Rp advertises 1.5 A (7.5 W), not 2 A (10 W)
- Y-cap ref des: rename C14 → C3 across all docs and schematic annotations
  to match BOM primary-section ordering; C14 remains the VBUS bypass cap on Sheet 05
- BUILD-SHEET-02 class table: correct IEEE 802.3af classes 0–3 with accurate
  power limits; remove non-existent "Class 4" row and misleading 802.3at note
- BOM: add F1 (2 A PPTC resettable fuse) for VBUS over-current protection,
  with procurement note covering TPS25940 eFuse as active alternative

Co-Authored-By: Claude Sonnet 4.6 <noreply@anthropic.com>
Other:
- note added: "SECONDARY SIDE (isolated 5 V rail) ──────────────────────────────────── Place here: • T1 secondary winding → D4 anode • D4: SS34 Schottky 60 V / 3 A — secondary rectifier Cathode → +5V rail • C10: 220 µF / 16 V polymer low-ESR — main output bulk • C11–C13: 22 µF / 10 V X5R 1210 — additional output bulk • C3: 1 nF / 2 kV Y-cap — GND_POE to GND_SEC (isolation bridge) Place this straddling the isola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"
- note added: "──── ROUTE NOTES ──── • Primary side: keep V_POE loop (bridges → bulk cap → Si3402-B) area as small as possible — high di/dt • Switch node V_SW trace: short and fat (≥ 0.5 mm), avoid coupling to MDI or USB signals • Feedback path: keep optocoupler + TL431 traces short, away from switch node • Y-cap C3 must physically straddle the isolation cut line and connect between the two separate GND pours •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"
- note added: "════════ ISOLATION BARRIER ════════ ← 4 mm → Place a KiCad Zone Cut here on ALL layers Mark with a yellow courtyard line on silkscreen Y-cap C3 (1 nF / 2 kV) bridges GND_POE to GND here"
- note removed: "SECONDARY SIDE (isolated 5 V rail) ──────────────────────────────────── Place here: • T1 secondary winding → D4 anode • D4: SS34 Schottky 60 V / 3 A — secondary rectifier Cathode → +5V rail • C10: 220 µF / 16 V polymer low-ESR — main output bulk • C11–C13: 22 µF / 10 V X5R 1210 — additional output bulk • C14: 1 nF / 2 kV Y-cap — GND_POE to GND_SEC (isolation bridge) Place this straddling the isol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"
- note removed: "──── ROUTE NOTES ──── • Primary side: keep V_POE loop (bridges → bulk cap → Si3402-B) area as small as possible — high di/dt • Switch node V_SW trace: short and fat (≥ 0.5 mm), avoid coupling to MDI or USB signals • Feedback path: keep optocoupler + TL431 traces short, away from switch node • Y-cap C14 must physically straddle the isolation cut line and connect between the two separate GND pours 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"
- note removed: "════════ ISOLATION BARRIER ════════ ← 4 mm → Place a KiCad Zone Cut here on ALL layers Mark with a yellow courtyard line on silkscreen Y-cap C14 (1 nF / 2 kV) bridges GND_POE to GND here"
Changed lines of the file:
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@@
 		(effects (font (size 1.27 1.27)) (justify left top))
 	)
-	(text "════════ ISOLATION BARRIER ════════\n         ← 4 mm → \n Place a KiCad Zone Cut here on ALL layers\n Mark with a yellow courtyard line on silkscreen\n Y-cap C14 (1 nF / 2 kV) bridges GND_POE to GND here"
+	(text "════════ ISOLATION BARRIER ════════\n         ← 4 mm → \n Place a KiCad Zone Cut here on ALL layers\n Mark with a yellow courtyard line on silkscreen\n Y-cap C3 (1 nF / 2 kV) bridges GND_POE to GND here"
 		(exclude_from_sim no)
 		(at 106.68 55.88 0)
 		(effects (font (size 1.27 1.27) bold) (justify center top))
 	)
-	(text "SECONDARY SIDE (isolated 5 V rail)\n────────────────────────────────────\nPlace here:\n  • T1 secondary winding → D4 anode\n  • D4: SS34 Schottky 60 V / 3 A — secondary rectifier\n       Cathode → +5V rail\n  • C10: 220 µF / 16 V polymer low-ESR — main output bulk\n  • C11–C13: 22 µF / 10 V X5R 1210 — additional output bulk\n  • C14: 1 nF / 2 kV Y-cap — GND_POE to GND_SEC (isolation bridge)\n         Place this straddling the isolation barrier line\n  • U6: PC817B optocoupler\n         LED side (pins 1-2): anode via R_OPT to +5V,\n                              cathode to TL431 anode\n         Transistor side (pins 3-4): collector to Si3402-B FB pin,\n                                     emitter to GND_POE\n  • U7: TL431 shunt regulator\n         REF pin → resistor divider from +5V to GND_SEC\n         R_UPPER (10 kΩ) from +5V to REF\n         R_LOWER (10 kΩ) from REF to GND_SEC → Vout = 5.0 V\n         ANODE → GND_SEC\n         CATHODE → optocoupler LED cathode\n  • R_OPT: 560 Ω 0402 — optocoupler LED current limit\n  • Snubber across T1 primary: 220 Ω + 470 pF in series\n    (place on primary side, across switching node and VDD)"
+	(text "SECONDARY SIDE (isolated 5 V rail)\n────────────────────────────────────\nPlace here:\n  • T1 secondary winding → D4 anode\n  • D4: SS34 Schottky 60 V / 3 A — secondary rectifier\n       Cathode → +5V rail\n  • C10: 220 µF / 16 V polymer low-ESR — main output bulk\n  • C11–C13: 22 µF / 10 V X5R 1210 — additional output bulk\n  • C3: 1 nF / 2 kV Y-cap — GND_POE to GND_SEC (isolation bridge)\n         Place this straddling the isolation barrier line\n  • U6: PC817B optocoupler\n         LED side (pins 1-2): anode via R_OPT to +5V,\n                              cathode to TL431 anode\n         Transistor side (pins 3-4): collector to Si3402-B FB pin,\n                                     emitter to GND_POE\n  • U7: TL431 shunt regulator\n         REF pin → resistor divider from +5V to GND_SEC\n         R_UPPER (10 kΩ) from +5V to REF\n         R_LOWER (10 kΩ) from REF to GND_SEC → Vout = 5.0 V\n         ANODE → GND_SEC\n         CATHODE → optocoupler LED cathode\n  • R_OPT: 560 Ω 0402 — optocoupler LED current limit\n  • Snubber across T1 primary: 220 Ω + 470 pF in series\n    (place on primary side, across switching node and VDD)"
 		(exclude_from_sim no)
 		(at 127.0 25.4 0)
 		(effects (font (size 1.27 1.27)) (justify left top))
 	)
-	(text "──── ROUTE NOTES ────\n• Primary side: keep V_POE loop (bridges → bulk cap → Si3402-B) area as small as possible — high di/dt\n• Switch node V_SW trace: short and fat (≥ 0.5 mm), avoid coupling to MDI or USB signals\n• Feedback path: keep optocoupler + TL431 traces short, away from switch node\n• Y-cap C14 must physically straddle the isolation cut line and connect between the two separate GND pours\n• Output bulk caps C10–C13 go as close to the +5V hierarchical label as possible\n• Add stitching vias around primary GND pour perimeter to tie all primary GND copper together"
+	(text "──── ROUTE NOTES ────\n• Primary side: keep V_POE loop (bridges → bulk cap → Si3402-B) area as small as possible — high di/dt\n• Switch node V_SW trace: short and fat (≥ 0.5 mm), avoid coupling to MDI or USB signals\n• Feedback path: keep optocoupler + TL431 traces short, away from switch node\n• Y-cap C3 must physically straddle the isolation cut line and connect between the two separate GND pours\n• Output bulk caps C10–C13 go as close to the +5V hierarchical label as possible\n• Add stitching vias around primary GND pour perimeter to tie all primary GND copper together"
 		(exclude_from_sim no)
 		(at 25.4 205.74 0)

Commit message: Add gh0stee.com branding to all title blocks and README
Added (company "gh0stee.com") to the KiCad title_block of all six
schematics (root + Sheets 01–05) and the PCB file so the company name
appears in every printed/exported title block. Added a byline link to
README.md below the project description.

Co-Authored-By: Claude Sonnet 4.6 <noreply@anthropic.com>
Other:
- company: (none) -> gh0stee.com
Changed lines of the file:
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@@
 		(date "2026-05-10")
 		(rev "A")
+		(company "gh0stee.com")
 		(comment 1 "Schottky bridges → Si3402-B PoE PD → flyback T1 → 5 V / 2 A secondary rail")
 		(comment 2 "Primary side LEFT of barrier | Secondary side RIGHT of barrier")
