File: hardware/03_Bias_Rails.kicad_sch (KiCad schematic)
At the start: 0 parts

Commit message: Add gh0stee.com branding to all title blocks and README
Added (company "gh0stee.com") to the KiCad title_block of all six
schematics (root + Sheets 01–05) and the PCB file so the company name
appears in every printed/exported title block. Added a byline link to
README.md below the project description.

Co-Authored-By: Claude Sonnet 4.6 <noreply@anthropic.com>
Other:
- company: (none) -> gh0stee.com
Changed lines of the file:
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@@
 		(date "2026-05-11")
 		(rev "A")
+		(company "gh0stee.com")
 		(comment 1 "+3V3 (U4 AP2112K-3.3) and +1V0 (U5 RT9013-10GB) LDOs from the isolated 5 V rail")
 		(comment 2 "Both outputs feed Sheet 04 (RTL8153B I/O ring and core)")
