File: hardware/04_RTL8153B_Bridge.kicad_sch (KiCad schematic)
At the start: 0 parts

Commit message: Add gh0stee.com branding to all title blocks and README
Added (company "gh0stee.com") to the KiCad title_block of all six
schematics (root + Sheets 01–05) and the PCB file so the company name
appears in every printed/exported title block. Added a byline link to
README.md below the project description.

Co-Authored-By: Claude Sonnet 4.6 <noreply@anthropic.com>
Other:
- company: (none) -> gh0stee.com
Changed lines of the file:
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@@
 		(date "2026-05-11")
 		(rev "A")
+		(company "gh0stee.com")
 		(comment 1 "Realtek RTL8153B USB 3.0 ↔ Gigabit Ethernet controller (~60 pins)")
 		(comment 2 "EEPROM U3 (93C46) | 25 MHz crystal Y1 | Reset SW1 | LED drivers")
