File: hardware/05_USBC_Connector.kicad_sch (KiCad schematic)
At the start: 0 parts

Commit message: Add gh0stee.com branding to all title blocks and README
Added (company "gh0stee.com") to the KiCad title_block of all six
schematics (root + Sheets 01–05) and the PCB file so the company name
appears in every printed/exported title block. Added a byline link to
README.md below the project description.

Co-Authored-By: Claude Sonnet 4.6 <noreply@anthropic.com>
Other:
- company: (none) -> gh0stee.com
Changed lines of the file:
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@@
 		(date "2026-05-11")
 		(rev "A")
+		(company "gh0stee.com")
 		(comment 1 "USB-C receptacle J2, CC Rp pull-ups, VBUS bulk, ESD array U9, SS AC-coupling, PPTC fuse F1")
 		(comment 2 "Source role: 5 V output. CC Rp = 22 kΩ → advertises 1.5 A (7.5 W)")
